Commit message: add the gps sensor!

File: src/robot_simulator/robot_description/urdf/robot.xacro (robot description, xacro)
@@ -157,4 +157,5 @@
   </collision>
 </link>
+<!-- 添加imu连接 -->
 <joint name="imu_fixed_joint" type="fixed">
   <origin xyz="0.0 0.0 0.923475" rpy="0 0 0"/>
@@ -182,3 +183,33 @@
   </collision>
 </link>
+<link name="gps_link">
+  <inertial>
+    <mass value="0.1"/>
+    <origin xyz="0 0 0" />
+    <inertia ixx="0.01" iyy="0.01" izz="0.01" ixy="0.01" ixz="0.01" iyz="0.01"/>
+  </inertial>
+  <visual>
+    <geometry>
+      <sphere radius="0.01"/>
+    </geometry>
+    <material name="silver"/>
+  </visual>
+  <collision>
+    <geometry>
+      <sphere radius="0.1"/>
+    </geometry>
+  </collision>
+  <sensor name="gps_sensor" type="gps">
+    <update_rate>1.0</update_rate>
+    <visualize>true</visualize>
+    <gps>
+      <position>0 0 0</position>
+    </gps>
+  </sensor>
+</link>
+<joint name="gps_link_joint" type="fixed">
+  <parent link="base_link" />
+  <child link="gps_link" />
+  <origin xyz="0.0 0.0 0.1" rpy="0 0 0" />  <!-- 适当设置位置 -->
+</joint>
 </robot>

Commit message: change urdf , add submodule of velodyne

File: src/robot_simulator/robot_description/urdf/robot.xacro (robot description, xacro)
@@ -49,7 +49,7 @@
   min_range="0.5"
   max_range="130"
-  gpu="false"
+  gpu="true"
 >
-  <origin xyz="0.0 0.0 1.103475" rpy="0 0 0" />
+  <origin xyz="0.0 0.0 1.153" rpy="0 0 0" />
 </xacro:VLP-16>
 <joint name="back_right_wheel_joint" type="continuous">
@@ -211,5 +211,5 @@
   <parent link="base_link" />
   <child link="gps_link" />
-  <origin xyz="0.0 0.0 0.1" rpy="0 0 0" />  <!-- 适当设置位置 -->
+  <origin xyz="0.0 0.0 0.8" rpy="0 0 0" />  <!-- 适当设置位置 -->
 </joint>
 </robot>

Commit message: add the solar world map!

File: src/robot_simulator/robot_description/urdf/robot.xacro (robot description, xacro)
@@ -211,5 +211,5 @@
   <parent link="base_link" />
   <child link="gps_link" />
-  <origin xyz="0.0 0.0 0.1" rpy="0 0 0" />  <!-- 适当设置位置 -->
+  <origin xyz="0.0 0.0 0.9" rpy="0 0 0" />  <!-- 适当设置位置 -->
 </joint>
 </robot>

Commit message: update simulator environment!

File: src/robot_simulator/robot_description/urdf/robot.xacro (robot description, xacro)
@@ -211,9 +211,5 @@
   <parent link="base_link" />
   <child link="gps_link" />
-<<<<<<< HEAD
   <origin xyz="0.0 0.0 0.9" rpy="0 0 0" />  <!-- 适当设置位置 -->
-=======
-  <origin xyz="0.0 0.0 0.8" rpy="0 0 0" />  <!-- 适当设置位置 -->
->>>>>>> 357842948654f229d842b60ac3a98132e96878e8
 </joint>
 </robot>
