Commit message: realize waypoints nav

File: src/robot_simulator/robot_description/urdf/robot_mecanum.xacro (robot description, xacro)
@@ -56,5 +56,5 @@
 >
   <!-- <origin xyz="0.0 0.0 1.153" rpy="0 0 0" /> -->
-  <origin xyz="0.2 0.0 0.9" rpy="0 0.3 0" />
+  <origin xyz="0.2 0.0 0.6" rpy="0 0 0" />
 </xacro:VLP-16>
 <!-- 加载驱动轮模型  -->
